File: hardware/MainBoard/TrafficLight.kicad_sch (KiCad schematic)
At the start: 69 parts, among them J1 Screw_Terminal_01x09, J10 Screw_Terminal_01x07, J11 Screw_Terminal_01x09, J12 Screw_Terminal_01x07, J13 Screw_Terminal_01x09, J14 Screw_Terminal_01x07, J15 Screw_Terminal_01x09, J16 Screw_Terminal_01x07, J17 Screw_Terminal_01x09, J18 Screw_Terminal_01x07, J19 Screw_Terminal_01x09, J2 Screw_Terminal_01x07, J20 Screw_Terminal_01x07, J21 Screw_Terminal_01x09, J22 Screw_Terminal_01x07, J23 Screw_Terminal_01x09, J3 Screw_Terminal_01x06, J4 Screw_Terminal_01x07, J5 Screw_Terminal_01x09, J6 Screw_Terminal_01x07, J7 Screw_Terminal_01x09, J8 Screw_Terminal_01x07, J9 Screw_Terminal_01x09, U1 ESP32-DevKitC, U10 74HC595, U11 74HC595, U12 74HC595, U13 74HC595, U3 74HC595, U4 74HC595, U5 74HC595, U6 74HC595, U7 74HC595, U8 74HC595, U9 74HC595

Commit message: Electrical Cabinet
Started diagram for electrical cabinet and overall wiring schema
Parts:
- removed J1, J11, J13, J15, J17, J19, J21, J23, J5, J7, J9: Screw_Terminal_01x09, symbol Connector:Screw_Terminal_01x09
- removed J10, J12, J14, J16, J18, J2, J20, J22, J4, J6, J8: Screw_Terminal_01x07, symbol Connector:Screw_Terminal_01x07
- removed OC1, OC10, OC11, OC12, OC13, OC14, OC15, OC16, OC17, OC18, OC19, OC2, OC20, OC21, OC22, OC3, OC4, OC5, OC6, OC7, OC8, OC9: PC847, PCM_Package_DIP_AKL:DIP-16_W7.62mm_LongPads, symbol PCM_Optocoupler_AKL:PC847
- removed R1, R10, R11, R2, R3, R4, R5, R6, R7, R8, R9: R, symbol Device:R
- removed U10, U11, U12, U13, U3, U4, U5, U6, U7, U8, U9: 74HC595, symbol 74xx:74HC595
Other:
- note removed: "500-10"
- note removed: "500-11"
- note removed: "500-2"
- note removed: "500-3"
- note removed: "500-4"
- note removed: "500-5"
- note removed: "500-6"
- note removed: "500-7"
- note removed: "500-8"
- note removed: "500-9"
- note removed: "550-10"
- note removed: "550-11"
- note removed: "550-2"
- note removed: "550-3"
- note removed: "550-4"
- note removed: "550-5"
- note removed: "550-6"
- note removed: "550-7"
- note removed: "550-8"
- note removed: "550-9"
- note removed: "7400-1"
- note removed: "7400-10"
- note removed: "7400-2"
- note removed: "7400-3"
- note removed: "7400-4"
- note removed: "7400-5"
- note removed: "7400-6"
- note removed: "7400-7"
- note removed: "7400-8"
- note removed: "7400-9"
- moved on the sheet: 1000BLOCK, U1
