File: hardware/RelayBoard/TrafficLight_RelayModule.kicad_pcb (KiCad board)
At the start: 2 copper layers, 28 parts, among them J1 Screw_Terminal_01x09, J2 Screw_Terminal_01x06, K1 G3MB-202P DC5, K2 G3MB-202P DC5, K3 G3MB-202P DC5, K4 G3MB-202P DC5, K5 G3MB-202P DC5, K6 G3MB-202P DC5, K7 G3MB-202P DC5, K8 G3MB-202P DC5, U1 TPIC6B595N

Commit message: Electrical Cabinet
Started diagram for electrical cabinet and overall wiring schema
Other:
- board outline added: 76 x 76 mm
Changed lines of the file:
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@@
 		(filling no)
 		(pcbplotparams
-			(layerselection 0x00000000_00000000_55555555_5755f5ff)
+			(layerselection 0x00000000_00000000_55555555_57557573)
 			(plot_on_all_layers_selection 0x00000000_00000000_00000000_00000000)
 			(disableapertmacros no)
@@
 			(outputformat 1)
 			(mirror no)
-			(drillshape 1)
+			(drillshape 0)
 			(scaleselection 1)
-			(outputdirectory "")
+			(outputdirectory "Gerber/")
 		)
 	)
@@
 		(embedded_fonts no)
 	)
+	(gr_rect
+		(start 26.5 16.5)
+		(end 102.5 92.5)
+		(stroke
+			(width 0.05)
+			(type default)
+		)
+		(fill no)
+		(layer "Edge.Cuts")
+	)
 	(segment
 		(start 30.786 35)
@@
 	)
 	(segment
+		(start 89.582 84.96)
+		(end 89.582 82.582)
+		(width 0.2)
+		(layer "F.Cu")
+		(net "Net-(J2-Pin_6)")
+	)
+	(segment
 		(start 72.2 68.5)
 		(end 85.2 68.5)
@@
 	)
 	(segment
-		(start 86.32 67.38)
-		(end 90 71.06)
+		(start 88.35 79.248)
+		(end 89.97 79.248)
 		(width 0.2)
 		(layer "F.Cu")
@@
 	)
 	(segment
-		(start 89.582 84.96)
-		(end 89.582 79.624)
+		(start 86.32 67.38)
+		(end 89.97 71.03)
 		(width 0.2)
 		(layer "F.Cu")
@@
 	)
 	(segment
-		(start 90 71.06)
-		(end 90 78.928)
+		(start 89.97 79.248)
+		(end 89.97 71.03)
 		(width 0.2)
 		(layer "F.Cu")
@@
 	)
 	(segment
-		(start 85.2 68.5)
-		(end 86.32 67.38)
+		(start 89.582 82.582)
+		(end 89.97 82.194)
 		(width 0.2)
 		(layer "F.Cu")
@@
 	)
 	(segment
-		(start 89.582 79.624)
-		(end 89.958 79.248)
+		(start 85.2 68.5)
+		(end 86.32 67.38)
 		(width 0.2)
 		(layer "F.Cu")
@@
 	)
 	(segment
-		(start 88.35 79.248)
-		(end 89.958 79.248)
+		(start 89.97 82.194)
+		(end 89.97 79.248)
 		(width 0.2)
 		(layer "F.Cu")
